Commit message: 导航与建图功能完成，等待实机测试

File: src/cleanbot_control/config/cleanbot_real.urdf.xacro (robot description, xacro)
@@ -1,8 +1,10 @@
 <?xml version="1.0"?>
-<robot xmlns:xacro="http://www.ros.org/wiki/xacro" name="cleanbot">
+<robot xmlns:xacro="http://ros.org/wiki/xacro" name="cleanbot">
     <!-- 包含真实硬件的ros2_control配置 -->
     <xacro:include filename="$(find cleanbot_control)/config/cleanbot_real.ros2_control.xacro"/>
-    <!-- 基础结构 -->
+    <!-- ======================== 基础结构 ======================== -->
+    <!-- 地面投影点 -->
     <link name="base_footprint"/>
+    <!-- 机器人主体 -->
     <link name="base_link">
         <visual>
@@ -29,4 +31,5 @@
         <origin xyz="0 0 0.06" rpy="0 0 0"/>
     </joint>
+    <!-- ======================== 轮子 ======================== -->
     <!-- 左轮 -->
     <link name="left_wheel_link">
@@ -85,6 +88,25 @@
         <axis xyz="0 1 0"/>
     </joint>
+    <!-- ======================== 传感器 ======================== -->
     <!-- IMU -->
-    <link name="imu_link"/>
+    <link name="imu_link">
+        <visual>
+            <geometry>
+                <box size="0.02 0.02 0.02"/>
+            </geometry>
+            <material name="blue">
+                <color rgba="0 0 1 0.5"/>
+            </material>
+        </visual>
+        <collision>
+            <geometry>
+                <box size="0.02 0.02 0.02"/>
+            </geometry>
+        </collision>
+        <inertial>
+            <mass value="0.01"/>
+            <inertia ixx="0.00001" ixy="0.0" ixz="0.0" iyy="0.00001" iyz="0.0" izz="0.00001"/>
+        </inertial>
+    </link>
     <joint name="imu_joint" type="fixed">
         <parent link="base_link"/>
@@ -92,5 +114,55 @@
         <origin xyz="0 0 0.02" rpy="0 0 0"/>
     </joint>
-    <!-- 调用ros2_control宏 -->
+    <!-- 激光雷达支撑杆 -->
+    <link name="laser_support_link">
+        <visual>
+            <geometry>
+                <cylinder radius="0.01" length="0.08"/>
+            </geometry>
+            <material name="grey">
+                <color rgba="0.5 0.5 0.5 1.0"/>
+            </material>
+        </visual>
+        <collision>
+            <geometry>
+                <cylinder radius="0.01" length="0.08"/>
+            </geometry>
+        </collision>
+        <inertial>
+            <mass value="0.05"/>
+            <inertia ixx="0.0001" ixy="0.0" ixz="0.0" iyy="0.0001" iyz="0.0" izz="0.00001"/>
+        </inertial>
+    </link>
+    <joint name="laser_support_joint" type="fixed">
+        <parent link="base_link"/>
+        <child link="laser_support_link"/>
+        <origin xyz="0 0 0.10" rpy="0 0 0"/>
+    </joint>
+    <!-- 激光雷达 (RPLidar A1) -->
+    <link name="laser">
+        <visual>
+            <geometry>
+                <cylinder radius="0.035" length="0.04"/>
+            </geometry>
+            <material name="black">
+                <color rgba="0 0 0 1.0"/>
+            </material>
+        </visual>
+        <collision>
+            <geometry>
+                <cylinder radius="0.035" length="0.04"/>
+            </geometry>
+        </collision>
+        <inertial>
+            <mass value="0.15"/>
+            <inertia ixx="0.0001" ixy="0.0" ixz="0.0" iyy="0.0001" iyz="0.0" izz="0.0001"/>
+        </inertial>
+    </link>
+    <joint name="laser_joint" type="fixed">
+        <parent link="laser_support_link"/>
+        <child link="laser"/>
+        <origin xyz="0 0 0.06" rpy="0 0 0"/>
+    </joint>
+    <!-- ======================== ros2_control ======================== -->
     <xacro:cleanbot_ros2_control_real/>
 </robot>

Commit message: 修正实机urdf

File: src/cleanbot_control/config/cleanbot_real.urdf.xacro (robot description, xacro)
@@ -112,5 +112,5 @@
         <parent link="base_link"/>
         <child link="imu_link"/>
-        <origin xyz="0 0 0.02" rpy="0 0 0"/>
+        <origin xyz="0.08 -0.04 0.02" rpy="0 0 0"/>
     </joint>
     <!-- 激光雷达支撑杆 -->
@@ -137,5 +137,5 @@
         <parent link="base_link"/>
         <child link="laser_support_link"/>
-        <origin xyz="0 0 0.10" rpy="0 0 0"/>
+        <origin xyz="0.10 0 0.10" rpy="0 0 3.14"/>
     </joint>
     <!-- 激光雷达 (RPLidar A1) -->
